Commit message: changes in robot design and world and creating docker and compose for GUI

File: src/minebot_playground/urdf/naviq.urdf (robot description, URDF)
Before this commit: robot naviq, 7 links, 6 joints
Links:
- removed link caster_wheel
- added link left_track; visual box size=0.6 0.12 0.18
- added link right_track; visual box size=0.6 0.12 0.18
- link camera_link: mass 0.05 -> 0.01; geometry collision box size=0.04 0.08 0.04; visual box size=0.04 0.08 0.04
- link carbon_monoxide_gas_sensor: mass 0.1 -> None; geometry visual box size=0.18 0.1 0.02
- link general_gas_sensor: mass 0.1 -> None; geometry visual box size=0.18 0.1 0.02
- link left_wheel: geometry collision cylinder length=0.05 radius=0.1
- link right_wheel: geometry collision cylinder length=0.05 radius=0.1
Joints:
- removed joint base_right_caster_wheel
- added joint base_to_left_track: type fixed, parent base_link, child left_track, origin xyz=0 0.25 0.1
- added joint base_to_right_track: type fixed, parent base_link, child right_track, origin xyz=0 -0.25 0.1
- joint base_camera_joint: origin xyz=0.31 0 0.21 rpy=0 0 0 -> xyz=0.31 0 0.26 rpy=0 0 0
- joint base_carbon_monoxide_gas_sensor: origin xyz=0 -0.12 0.22 rpy=0 0 0 -> xyz=0.10 -0.12 0.26 rpy=0 0 0
- joint base_general_gas_sensor: origin xyz=0 0.12 0.22 rpy=0 0 0 -> xyz=0.10 0.12 0.26 rpy=0 0 0
- joint base_left_wheel_joint: origin xyz=-0.15 0.225 0 rpy=0 0 0 -> xyz=0 0.225 0.1 rpy=0 0 0
- joint base_right_wheel_joint: origin xyz=-0.15 -0.225 0 rpy=0 0 0 -> xyz=0 -0.225 0.1 rpy=0 0 0
